File: 80col_64k.kicad_sch (KiCad schematic)
At the start: 17 parts, among them J1 Conn_02x30_Counter_Clockwise, U1 4464, U2 4464, U3 74LS245, U4 74LS374, U5 74LS14

Commit message: add title block info
Other:
- company: (none) -> Bradley Bell
- title: (none) -> Apple IIe 80 column/64k memory expansion card
Changed lines of the file:
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@@
 (kicad_sch (version 20230121) (generator eeschema)
   (paper "USLetter")
+  (title_block
+    (title "Apple IIe 80 column/64k memory expansion card")
+    (date "2024-02-17")
+    (rev "0")
+    (company "Bradley Bell")
+  )
   (junction (at 222.25 114.3) (diameter 0) (color 0 0 0 0)
   )
